Commit message: Hand controller URDF created. simulation function using rbdl created. Added loop closure in dynamics_model.cpp

File: hand_controller/urdf/hand_controller.urdf (robot description, URDF)
Before this commit: robot hand_controller, 4 links, 3 joints
Links:
- removed link link0
- removed link link1
- removed link link2
- added link base_link, mass 0.5; visual cylinder length=0.02 radius=0.08
- added link body_link, mass 2.5; collision box size=0.08 0.06 0.06; collision box size=0.15 0.15 0.12
- added link capstan_link, mass 0.25; collision box size=0.1 0.02 0.02; visual box size=0.1 0.02 0.02
- added link elbow_frame_link1, mass 0.25
- added link elbow_frame_link2, mass 0.25
- added link elbow_link, mass 0.25; collision box size=0.04 0.04 0.3; visual box size=0.04 0.04 0.3
- added link forearm_frame_link
- added link forearm_link, mass 0.25; collision box size=0.5 0.04 0.04; visual box size=0.5 0.04 0.04
- added link gripper_link
- added link support_link, mass 0.25; collision box size=0.02 0.02 0.3; visual box size=0.02 0.02 0.3
- added link wrist_link1, mass 0.25; visual box size=0.02 0.02 0.15; visual box size=0.15 0.02 0.02
- added link wrist_link2, mass 0.25; visual box size=0.02 0.02 0.12; visual box size=0.12 0.02 0.02
- added link wrist_link3, mass 0.25; visual box size=0.02 0.02 0.08; visual box size=0.08 0.02 0.02
Joints:
- removed joint joint1
- removed joint joint2
- added joint backelbow_joint: type revolute, parent support_link, child forearm_link, origin xyz=0 -0.02 0.3 rpy=0 0 0, axis 0 1 0, limit lower=-3.14 upper=3.14 effort=0 velocity=0
- added joint base_joint: type revolute, parent base_link, child body_link, origin xyz=0 0 0.01 rpy=0 0 0, axis 0 0 1, limit lower=-3.14 upper=3.14 effort=0 velocity=0
- added joint capstan_joint: type revolute, parent body_link, child capstan_link, origin xyz=0.04 0.03 0.15 rpy=0 0 0, axis 0 1 0, limit lower=-3.14 upper=3.14 effort=0 velocity=0
- added joint elbow_frame_joint1: type fixed, parent elbow_link, child elbow_frame_link1, origin xyz=0 0 0.3 rpy=0 0 0
- added joint elbow_frame_joint2: type fixed, parent forearm_link, child elbow_frame_link2, origin xyz=-0.18 -0.04 0 rpy=0 0 0
- added joint forearm_joint: type fixed, parent forearm_link, child forearm_frame_link, origin xyz=-0.5 -0.02 0.02 rpy=0 0 0
- added joint gripper_joint: type fixed, parent wrist_link3, child gripper_link, origin xyz=0.08 0 0.08 rpy=0 -1.57 -3.14
- added joint shoulder_joint: type revolute, parent body_link, child elbow_link, origin xyz=-0.04 -0.03 0.15 rpy=0 0 0, axis 0 1 0, limit lower=-3.14 upper=3.14 effort=0 velocity=0
- added joint support_joint: type revolute, parent capstan_link, child support_link, origin xyz=0.1 0 0 rpy=0 0 0, axis 0 1 0, limit lower=-3.14 upper=3.14 effort=0 velocity=0
- added joint wrist_joint1: type revolute, parent forearm_frame_link, child wrist_link1, origin xyz=0 0 0 rpy=0 0 0, axis 0 0 1, limit lower=-3.14 upper=3.14 effort=0 velocity=0
- added joint wrist_joint2: type revolute, parent wrist_link1, child wrist_link2, origin xyz=0.15 0 0.15 rpy=0 1.57 -3.14, axis 0 0 1, limit lower=-3.14 upper=3.14 effort=0 velocity=0
- added joint wrist_joint3: type revolute, parent wrist_link2, child wrist_link3, origin xyz=0.12 0 0.12 rpy=0 1.57 -3.14, axis 0 0 1, limit lower=-3.14 upper=3.14 effort=0 velocity=0
- joint dummy_joint: child link0 -> base_link

Commit message: Working on constraint

File: hand_controller/urdf/hand_controller.urdf (robot description, URDF)
Before this commit: robot hand_controller, 14 links, 13 joints
Links:
- removed link elbow_frame_link1
- removed link elbow_frame_link2
- added link elbow_constraint_frame_link, mass 0.25
- added link forearm_constraint_frame_link, mass 0.25
Joints:
- joint elbow_frame_joint1: child elbow_frame_link1 -> elbow_constraint_frame_link
- joint elbow_frame_joint2: child elbow_frame_link2 -> forearm_constraint_frame_link
